File: Kicad_8_files/CANbardo.kicad_pcb (KiCad board)
At the start: 4 copper layers, 56 x 70 mm, 103 parts, among them J1 USB_C_Receptacle_USB2.0, J3 DE9_Plug_MountingHoles, J4 DE9_Plug_MountingHoles, J5 Conn_01x08_Pin, Q1 2N7002, Q2 2N7002, SW1 FSM4JSMAATR., U1 AC37S, U13 ATSAME70N20B-AN, U2 MCP2558FD-xSN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

Commit message: Updated LED resistors
LED resistors updated to match intensity.
Version updated from 1.0 to 1.1
Parts:
- R11, R12, R5: value 200R -> 2.7k
- R13, R16, R32: value 200R -> 390R
- R14, R19: value 200R -> 620R
